File: Sis. de iluminacion.kicad_pcb (KiCad board)
At the start: 2 copper layers, 86.8 x 98.1 mm, 48 parts, among them J1 Screw_Terminal_01x02, J10 Screw_Terminal_01x02, J11 Screw_Terminal_01x02, J12 Screw_Terminal_01x02, J3 Screw_Terminal_01x02, J4 Conn_01x04, J5 Screw_Terminal_01x02, J7 Screw_Terminal_01x02, J8 Screw_Terminal_01x02, J9 Screw_Terminal_01x02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

Commit message: Add files via upload
Parts:
- moved Q7 0.56 mm to (219.0, 129.6)
- moved D18 0.56 mm to (213.6, 78.7)
- moved D19 0.56 mm to (214.4, 105.2)
- moved D22 0.56 mm to (214.1, 126.4)
- moved J10 0.56 mm to (184.6, 74.5)
- moved J11 0.56 mm to (184.6, 99.0)
- moved J12 0.56 mm to (184.9, 123.2)
- moved J5 0.56 mm to (184.4, 82.7)
- moved J7 0.56 mm to (184.7, 106.9)
- moved K11 0.56 mm to (209.5, 123.5)
- moved K9 0.56 mm to (209.2, 75.4)
- moved R28 0.56 mm to (231.2, 86.0)
- moved R33 0.56 mm to (223.6, 98.2)
- moved C1 0.56 mm to (257.3, 55.2)
- moved D15 0.56 mm to (214.3, 57.7)
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Routing:
- net +12V: track 398.2 -> 400.0 mm

Commit message: Add files via upload
Parts:
- moved R17 1.85 mm to (238.4, 65.5)
- moved R16 0.90 mm to (240.3, 68.7)
Routing:
- net Net-(J4-Pin_3): track 6.63 -> 8.13 mm
- net GIOP32: track 29.3 -> 28.4 mm
- net +5V: track 167.9 -> 168.6 mm

Commit message: Add files via upload
Parts:
- J4: footprint Connector_PinSocket_2.00mm:PinSocket_1x04_P2.00mm_Vertical -> Connector_PinSocket_2.54mm:PinSocket_1x04_P2.54mm_Vertical
- moved R17 14.6 mm to (252.0, 70.7)
- moved R16 14.6 mm to (253.9, 73.9)
- moved J4 14.4 mm to (259.0, 66.9)
Connections:
- J4 pad 2: GIOP33 -> GIOP22
- R16 pad 1: GIOP32 -> GIOP23
- R24 pad 1: GIOP34 -> GIOP35
- R28 pad 1: GIOP39 -> GIOP32
- R32 pad 1: GIOP35 -> GIOP33
- U1 pad 14: unconnected-(U1-GND-Pad14) -> GND
- U1 pad 32: unconnected-(U1-GND-Pad32) -> GND
- U1 pad 33: unconnected-(U1-IO21-Pad33) -> GIOP21
- U1 pad 36: unconnected-(U1-IO22-Pad36) -> GIOP22
- U1 pad 37: unconnected-(U1-IO23-Pad37) -> GIOP23
- U1 pad 38: unconnected-(U1-GND-Pad38) -> GND
- U1 pad 4: GIOP39 -> unconnected-(U1-SVN-Pad4)
Routing:
- net GIOP34: track 33.8 -> 0.00 mm
- net GIOP22: track 0.00 -> 25.6 mm
- net GND: track 55.2 -> 80.4 mm
- net GIOP33: track 39.2 -> 15.1 mm
- net GIOP32: track 28.4 -> 9.44 mm
- net GIOP35: track 20.1 -> 38.6 mm
- net GIOP23: track 0.00 -> 16.4 mm
- net +5V: track 168.6 -> 180.1 mm
- net GIOP39: track 5.10 -> 0.00 mm
- net +12V: track 400.0 -> 404.5 mm
- net Net-(J4-Pin_3): track 8.13 -> 7.43 mm
Other:
- board size 86.8 x 98.1 mm -> 88.9 x 98.1 mm

Commit message: Add files via upload
Parts:
- D16, D18, D20, D22: footprint Diode_SMD:D_0805_2012Metric -> Diode_SMD:D_SMA
- moved J4 20.5 mm to (238.6, 65.0), turned to 90 degrees
- moved R16 9.49 mm to (244.7, 71.4)
- moved R17 7.67 mm to (244.7, 68.3), turned to 180 degrees
- moved R32 5.56 mm to (228.2, 112.2), turned to 90 degrees
- moved D17 4.48 mm to (213.6, 85.9)
- moved U1 3.95 mm to (251.4, 98.0), turned to 90 degrees
- moved R28 3.59 mm to (228.8, 88.7)
- moved D19 3.36 mm to (213.9, 108.5)
- moved D21 3.30 mm to (214.4, 132.9)
- moved R30 2.95 mm to (213.4, 72.0)
- moved D15 2.81 mm to (214.0, 60.5)
- moved R27 1.48 mm to (213.6, 49.0)
- moved R34 1.37 mm to (213.6, 97.2)
- moved R38 1.27 mm to (214.1, 121.5)
- moved D20 1.06 mm to (213.6, 103.2)
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Connections:
- J4 pad 2: GIOP22 -> GIOP18
- R16 pad 1: GIOP23 -> GIOP19
- R24 pad 1: GIOP35 -> GIOP21
- R28 pad 1: GIOP32 -> GIOP22
- R32 pad 1: GIOP33 -> GIOP23
- R36 pad 1: GIOP18 -> GIOP33
- U1 pad 31: unconnected-(U1-IO19-Pad31) -> GIOP19
- U1 pad 5: GIOP34 -> unconnected-(U1-IO34-Pad5)
- U1 pad 6: GIOP35 -> unconnected-(U1-IO35-Pad6)
- U1 pad 7: GIOP32 -> unconnected-(U1-IO32-Pad7)
Routing:
- net GND: track 80.4 -> 0.00 mm
- net GIOP21: track 0.00 -> 51.1 mm
- net GIOP33: track 15.1 -> 59.0 mm
- net GIOP35: track 38.6 -> 0.00 mm
- net GIOP19: track 0.00 -> 37.4 mm
- net +5V: track 180.1 -> 152.5 mm
- net GIOP18: track 60.3 -> 38.5 mm
- net GIOP32: track 9.44 -> 0.00 mm
- net Net-(D17-A): track 8.77 -> 16.4 mm
- net GIOP22: track 25.6 -> 32.9 mm
- net +12V: track 404.5 -> 411.7 mm
- net Net-(D17-K): track 14.9 -> 21.9 mm
- net Net-(D19-A): track 8.37 -> 14.1 mm
- net Net-(D21-A): track 8.66 -> 14.0 mm
- net Net-(D15-A): track 9.27 -> 13.8 mm
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
Commit message: Add files via upload
Parts:
- removed U1: ESP32_DEVKITC, EESTN5:ESP32_DEVKITC
- added U2: ESP32_DEVKITC, EESTN5:ESP32S, F.Cu at (250.9, 100.3)
- moved J5 4.54 mm to (186.0, 87.0), turned to 90 degrees
- moved J4 1.88 mm to (237.5, 66.6)
- moved R17 1.85 mm to (244.9, 70.2)
- moved R16 1.85 mm to (244.9, 73.2)
- moved D21 1.44 mm to (215.8, 132.7)
- moved R36 1.44 mm to (233.4, 132.1)
- moved D17 1.44 mm to (215.0, 85.7)
- moved D18 1.44 mm to (214.6, 79.2)
- moved D20 1.44 mm to (215.0, 103.0)
- moved D22 1.44 mm to (215.5, 127.2)
- moved J10 1.44 mm to (186.0, 74.3)
- moved J11 1.44 mm to (186.0, 98.8)
- moved J3 1.44 mm to (186.0, 62.6)
- moved J7 1.44 mm to (186.1, 106.7)
- moved J8 1.44 mm to (186.0, 50.6)
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Connections:
- J5 pad 1: NO1 -> V1
- J5 pad 2: V1 -> NO1
Routing:
- net +5V: track 152.5 -> 205.1 mm
- net NO9: track 7.67 -> 14.9 mm
- net GIOP33: track 59.0 -> 52.0 mm
- net GIOP18: track 38.5 -> 40.8 mm
- net +12V: track 411.7 -> 409.6 mm
- net Net-(J4-Pin_3): track 6.43 -> 7.69 mm
- net GIOP22: track 32.9 -> 33.9 mm
- net GIOP19: track 37.4 -> 36.4 mm
- net GIOP23: track 14.1 -> 15.0 mm
- net Net-(D21-A): track 14.0 -> 14.6 mm
- net COM9: track 20.8 -> 20.2 mm

Commit message: Add files via upload
Parts:
- D15, D17, D19, D21: footprint LED_SMD:LED_0805_2012Metric -> LED_THT:LED_D3.0mm; moved to F.Cu
- moved D19 2.25 mm to (213.8, 110.0)
- moved D21 1.83 mm to (214.2, 133.5)
- moved D17 1.33 mm to (213.7, 85.6)
- moved D15 1.20 mm to (214.3, 60.7)
- moved Q6 0.99 mm to (220.6, 105.5)
- moved Q7 0.77 mm to (221.1, 129.8)
- moved C1 0.15 mm to (258.8, 55.9)
- moved D16 0.15 mm to (214.9, 54.7)
- moved J12 0.15 mm to (186.4, 122.8)
- moved J9 0.15 mm to (186.3, 130.1)
- moved K8 0.15 mm to (211.1, 50.6)
- moved K9 0.15 mm to (210.7, 75.0)
- moved R24 0.15 mm to (232.7, 62.2)
- moved R25 0.15 mm to (226.0, 49.7)
- moved R28 0.15 mm to (230.3, 88.4)
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Routing:
- net Net-(D15-K): track 17.5 -> 24.5 mm
- net Net-(D19-K): track 17.8 -> 22.5 mm
- net Net-(D21-K): track 18.5 -> 21.8 mm
- net Net-(D19-A): track 14.1 -> 15.7 mm
