File: Sis. de iluminacion.kicad_sch (KiCad schematic)
At the start: 48 parts, among them J1 Screw_Terminal_01x02, J2 Screw_Terminal_01x04, J3 Screw_Terminal_01x02, J5 Screw_Terminal_01x02, J7 Screw_Terminal_01x02, J9 Screw_Terminal_01x02, K10 Relay_DPDT, K11 Relay_DPDT, K8 Relay_DPDT, K9 Relay_DPDT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

Commit message: Rele wifi
Parts:
- removed J2: Screw_Terminal_01x04, TerminalBlock:TerminalBlock_MaiXu_MX126-5.0-04P_1x04_P5.00mm, symbol Connector:Screw_Terminal_01x04
- removed R26, R31, R35, R39: 10K, Resistor_SMD:R_0805_2012Metric, symbol Device:R
- added J10, J11, J12, J8: Screw_Terminal_01x02, TerminalBlock:TerminalBlock_MaiXu_MX126-5.0-02P_1x02_P5.00mm, symbol Connector:Screw_Terminal_01x02
- added J4: Conn_01x04, Connector_PinSocket_2.00mm:PinSocket_1x04_P2.00mm_Vertical, symbol Connector_Generic:Conn_01x04
- K10, K11, K8, K9: footprint Relay_THT:Relay_DPDT_Schrack-RT2-FormC_RM5mm -> Relay_THT:Relay_DPDT_Omron_G6A
- Q4: footprint Package_TO_SOT_THT:TO-92_Inline -> Package_TO_SOT_THT:TO-92_Wide
- R24, R28, R32, R36: value 1K -> 220
Connections:
- net +5V: now also U11.4, U12.4, U13.4, J4.1 (Pin_1)
- net GIOP18: now also R36.1; no longer R16.1, R17.2
- net GIOP34: now also R24.1; no longer R36.1
- net GND: now also J4.4 (Pin_4)
- net LED +: now also J3.2 (Pin_2); no longer J3.1 (Pin_1)
- net NO1: now also J5.1 (Pin_1); no longer J5.2 (Pin_2)
- net NO2: now also J7.1 (Pin_1); no longer J7.2 (Pin_2)
- net NO3: now also J9.1 (Pin_1); no longer J9.2 (Pin_2)
- net V1: now also J5.2 (Pin_2); no longer J5.1 (Pin_1)
- net V2: now also J7.2 (Pin_2); no longer J7.1 (Pin_1)
- net V3: now also J9.2 (Pin_2); no longer J9.1 (Pin_1)
- net COM10: now reaches K10.11
- net COM10: now also J11.2 (Pin_2)
- net NO10: now reaches K10.14
- net NO10: now also J11.1 (Pin_1)
- net at R16.2: now also R17.2, J4.3 (Pin_3)
- net COM9: now reaches K9.11
- net COM9: now also J10.2 (Pin_2)
- net NO9: now reaches K9.14
- net NO9: now also J10.1 (Pin_1)
- net COM11: now reaches K11.11
- net COM11: now also J12.2 (Pin_2)
- net NO11: now reaches K11.14
- net NO11: now also J12.1 (Pin_1)
- net GIOP39: now reaches U1.4 (SVN)
- net GIOP39: now also R28.1
- net GIOP35: now reaches U1.6 (IO35)
- net GIOP35: now also R32.1
- net GIOP32: now reaches U1.7 (IO32)
- net GIOP32: now also R16.1
- net GIOP33: now reaches U1.8 (IO33)
- net GIOP33: now also J4.2 (Pin_2)
- net COM: now reaches K8.11
- net COM: now also J8.2 (Pin_2)
- net NO: now reaches K8.14
- net NO: now also J8.1 (Pin_1)
- net 3.3V: no longer names the net of U1.1 (3V3)
- net 5V renamed 5V1
- net 5V1: now also J3.1 (Pin_1); no longer J3.2 (Pin_2)
- net GIOP21: no longer names the net of U1.33 (IO21)
- net GIOP21: no longer R32.1
- net GIOP26: no longer names the net of U1.10 (IO26)
- net GIOP26: no longer R24.1
- net GIOP5: no longer names the net of U1.29 (IO5)
- net GIOP5: no longer R28.1
- net NC: no longer names the net of K8.22
- no-connect marks 8 -> 0
Other:
- note added: "ESP32"
- note added: "REGULADOR"
- note added: "RELE"
- note added: "ULTRASONIDO"
- moved on the sheet: C1, C2, D15, D16, D17, D18, D19, D20, D21, D22, J1, J3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

Commit message: Add files via upload
Parts:
- J4: footprint Connector_PinSocket_2.00mm:PinSocket_1x04_P2.00mm_Vertical -> Connector_PinSocket_2.54mm:PinSocket_1x04_P2.54mm_Vertical
Connections:
- net GIOP32: now also R28.1; no longer R16.1
- net GIOP33: now also R32.1; no longer J4.2 (Pin_2)
- net GIOP34: no longer R24.1
- net GIOP35: now also R24.1; no longer R32.1
- net GND: now also U1.14 (GND), U1.32 (GND), U1.38 (GND)
- net GIOP21: now reaches U1.33 (IO21)
- net GIOP22: now reaches U1.36 (IO22)
- net GIOP22: now also J4.2 (Pin_2)
- net GIOP23: now reaches U1.37 (IO23)
- net GIOP23: now also R16.1
- net GIOP39: no longer names the net of U1.4 (SVN)
- net GIOP39: no longer R28.1

Commit message: Add files via upload
Parts:
- D16, D18, D20, D22: footprint Diode_SMD:D_0805_2012Metric -> Diode_SMD:D_SMA
Connections:
- net GIOP18: now also J4.2 (Pin_2); no longer R36.1
- net GIOP21: now also R24.1
- net GIOP22: now also R28.1; no longer J4.2 (Pin_2)
- net GIOP23: now also R32.1; no longer R16.1
- net GIOP33: now also R36.1; no longer R32.1
- net GIOP19: now reaches U1.31 (IO19)
- net GIOP19: now also R16.1
- net GIOP32: no longer names the net of U1.7 (IO32)
- net GIOP32: no longer R28.1
- net GIOP34: no longer names the net of U1.5 (IO34)
- net GIOP35: no longer names the net of U1.6 (IO35)
- net GIOP35: no longer R24.1
Changed lines of the file:
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@@
 	)
 	(global_label "GIOP18"
-		(shape input)
+		(shape output)
 		(at 271.78 49.53 0)
 		(fields_autoplaced yes)
@@
 		)
 	)
-	(global_label "GIOP33"
+	(global_label "GIOP19"
 		(shape output)
-		(at 243.84 46.99 180)
+		(at 271.78 46.99 0)
 		(fields_autoplaced yes)
 		(effects
@@
 				(size 1.27 1.27)
 			)
-			(justify right)
+			(justify left)
 		)
 		(property "Intersheetrefs" "${INTERSHEET_REFS}"
-			(at 233.9605 46.99 0)
+			(at 281.6595 46.99 0)
 			(effects
 				(font
 					(size 1.27 1.27)
 				)
-				(justify right)
+				(justify left)
 				(hide yes)
 			)
 		)
 	)
-	(global_label "GIOP22"
+	(global_label "GIOP18"
 		(shape output)
 		(at 144.78 30.48 180)
@@
 	)
 	(global_label "GIOP22"
-		(shape input)
+		(shape output)
 		(at 271.78 34.29 0)
 		(fields_autoplaced yes)
@@
 	)
 	(global_label "GIOP23"
-		(shape input)
+		(shape output)
 		(at 271.78 31.75 0)
 		(fields_autoplaced yes)
@@
 		)
 	)
-	(global_label "GIOP32"
-		(shape output)
-		(at 243.84 44.45 180)
-		(fields_autoplaced yes)
-		(effects
-			(font
-				(size 1.27 1.27)
-			)
-			(justify right)
-		)
-		(property "Intersheetrefs" "${INTERSHEET_REFS}"
-			(at 233.9605 44.45 0)
-			(effects
-				(font
-					(size 1.27 1.27)
-				)
-				(justify right)
-				(hide yes)
-			)
-		)
-	)
 	(global_label "GIOP21"
 		(shape output)
@@
 		)
 	)
-	(global_label "GIOP35"
-		(shape output)
-		(at 243.84 41.91 180)
-		(fields_autoplaced yes)
-		(effects
-			(font
-				(size 1.27 1.27)
-			)
-			(justify right)
-		)
-		(property "Intersheetrefs" "${INTERSHEET_REFS}"
-			(at 233.9605 41.91 0)
-			(effects
-				(font
-					(size 1.27 1.27)
-				)
-				(justify right)
-				(hide yes)
-			)
-		)
-	)
 	(global_label "NO2"
 		(shape input)
@@
 		)
 	)
-	(global_label "GIOP35"
+	(global_label "GIOP21"
 		(shape output)
 		(at 137.16 87.63 180)
@@
 		)
 	)
-	(global_label "GIOP33"
-		(shape input)
+	(global_label "GIOP23"
+		(shape output)
 		(at 22.86 111.76 180)
 		(fields_autoplaced yes)
@@
 		)
 	)
-	(global_label "GIOP32"
+	(global_label "GIOP22"
 		(shape output)
 		(at 22.86 49.53 180)
@@
 		)
 	)
-	(global_label "GIOP34"
-		(shape output)
-		(at 243.84 39.37 180)
-		(fields_autoplaced yes)
-		(effects
-			(font
-				(size 1.27 1.27)
-			)
-			(justify right)
-		)
-		(property "Intersheetrefs" "${INTERSHEET_REFS}"
-			(at 233.9605 39.37 0)
-			(effects
-				(font
-					(size 1.27 1.27)
-				)
-				(justify right)
-				(hide yes)
-			)
-		)
-	)
 	(global_label "LED +"
 		(shape input)
@@
 		)
 	)
-	(global_label "GIOP18"
-		(shape input)
+	(global_label "GIOP33"
+		(shape output)
 		(at 22.86 173.99 180)
 		(fields_autoplaced yes)
@@
 		)
 	)
-	(global_label "GIOP23"
+	(global_label "GIOP33"
+		(shape output)
+		(at 243.84 46.99 180)
+		(fields_autoplaced yes)
+		(effects
+			(font
+				(size 1.27 1.27)
+			)
+			(justify right)
+		)
+		(property "Intersheetrefs" "${INTERSHEET_REFS}"
+			(at 233.9605 46.99 0)
+			(effects
+				(font
+					(size 1.27 1.27)
+				)
+				(justify right)
+				(hide yes)
+			)
+		)
+	)
+	(global_label "GIOP19"
 		(shape input)
 		(at 127 34.29 180)
@@
 			)
 		)
-		(property "Footprint" "Diode_SMD:D_0805_2012Metric"
+		(property "Footprint" "Diode_SMD:D_SMA"
 			(at 64.77 38.1 0)
 			(effects
@@
 			)
 		)
-		(property "Footprint" "Diode_SMD:D_0805_2012Metric"
+		(property "Footprint" "Diode_SMD:D_SMA"
 			(at 64.77 162.56 0)
 			(effects
@@
 			)
 		)
-		(property "Footprint" "Diode_SMD:D_0805_2012Metric"
+		(property "Footprint" "Diode_SMD:D_SMA"
 			(at 179.07 76.2 0)
 			(effects
@@
 			)
 		)
-		(property "Footprint" "Diode_SMD:D_0805_2012Metric"
+		(property "Footprint" "Diode_SMD:D_SMA"
 			(at 64.77 100.33 0)
 			(effects

Commit message: Add files via upload
Parts:
- removed U1: ESP32_DEVKITC, EESTN5:ESP32_DEVKITC, symbol EESTN5:ESP32_DEVKITC
- added U2: ESP32_DEVKITC, EESTN5:ESP32S, symbol EESTN5:ESP32_DEVKITC
Connections:
- net +5V: now also U2.19 (5V)
- net GIOP18: now also U2.30 (IO18)
- net GIOP19: now also U2.31 (IO19)
- net GIOP21: now also U2.33 (IO21)
- net GIOP22: now also U2.36 (IO22)
- net GIOP23: now also U2.37 (IO23)
- net GIOP33: now also U2.8 (IO33)
- net GND: now also U2.14 (GND), U2.32 (GND), U2.38 (GND)
- net NO1: now also J5.2 (Pin_2); no longer J5.1 (Pin_1)
- net V1: now also J5.1 (Pin_1); no longer J5.2 (Pin_2)
